Commit message: FIx robot name in gazebo plugin

File: lbr_description/gazebo/lbr_gazebo.xacro (robot description, xacro)
@@ -1,10 +1,10 @@
 <?xml version="1.0"?>
 <robot xmlns:xacro="http://www.ros.org/wiki/xacro">
-    <xacro:macro name="lbr_gazebo" params="robot_name:=^|lbr">
+    <xacro:macro name="lbr_gazebo" params="robot_name:=^|lbr controllers_config_path:=^|'$(find lbr_description)/ros2_control/lbr_controllers.yaml'">
         <!-- ros_control-plugin -->
         <gazebo>
             <plugin name="gz_ros2_control::GazeboSimROS2ControlPlugin"
                 filename="gz_ros2_control-system">
-                <parameters>$(find lbr_description)/ros2_control/lbr_controllers.yaml</parameters>
+                <parameters>${controllers_config_path}</parameters>
                 <ros>
                     <namespace>/${robot_name}</namespace>

File: lbr_description/urdf/med7/med7.xacro (robot description, xacro)
@@ -12,4 +12,7 @@
         name="initial_joint_positions_path"
         default="$(find lbr_description)/ros2_control/initial_joint_positions.yaml" />
+    <xacro:arg
+        name="controllers_config_path"
+        default="$(find lbr_description)/ros2_control/lbr_controllers.yaml" />
     <!-- KDL requires a link without inertia / Gazebo requires a connection to world link or robot
     will tipple https://github.com/lbr-stack/lbr_fri_ros2_stack/issues/230 -->
@@ -26,4 +29,5 @@
         mode="$(arg mode)"
         system_config_path="$(arg system_config_path)"
-        initial_joint_positions_path="$(arg initial_joint_positions_path)" />
+        initial_joint_positions_path="$(arg initial_joint_positions_path)"
+        controllers_config_path="$(arg controllers_config_path)" />
 </robot>

File: lbr_description/urdf/med7/med7_description.xacro (robot description, xacro)
@@ -3,5 +3,5 @@
     <!-- robot as extracted via https://github.com/syuntoku14/fusion2urdf -->
     <xacro:macro name="med7"
-        params="robot_name:=^|lbr mode:=^|mock system_config_path:=^|'$(find lbr_description)/ros2_control/lbr_system_config.yaml' initial_joint_positions_path:=^|'$(find lbr_description)/ros2_control/initial_joint_positions.yaml'">
+        params="robot_name:=^|lbr mode:=^|mock system_config_path:=^|'$(find lbr_description)/ros2_control/lbr_system_config.yaml' initial_joint_positions_path:=^|'$(find lbr_description)/ros2_control/initial_joint_positions.yaml' controllers_config_path:=^|'$(find lbr_description)/ros2_control/lbr_controllers.yaml'">
         <!-- includes -->
         <xacro:include filename="$(find lbr_description)/gazebo/lbr_gazebo.xacro" />
@@ -16,5 +16,7 @@
         <xacro:property name="joint_friction" value="0.1" />
         <!-- macros for gazebo / mock / hardware -->
-        <xacro:lbr_gazebo robot_name="${robot_name}" />
+        <xacro:lbr_gazebo
+            robot_name="${robot_name}"
+            controllers_config_path="${controllers_config_path}" />
         <xacro:lbr_system_interface
             robot_name="${robot_name}"
